Commit message: ydlidar

File: src/robot-nav/description/robot.urdf.xacro (robot description, xacro)
@@ -10,3 +10,6 @@
         <xacro:include filename="gazebo_control.xacro" />
     </xacro:unless>
+    <xacro:include filename="lidar.xacro" />
+    <!-- <xacro:include filename="camera.xacro" /> -->
+    <xacro:include filename="depth_camera.xacro" />
 </robot>

File: src/robot-nav/description/robot_core.xacro (robot description, xacro)
@@ -14,4 +14,7 @@
     <material name="black">
         <color rgba="0.0 0.0 0.0 1.0" />
+    </material>
+    <material name="red">
+        <color rgba="1.0 0.0 0.0 1.0" />
     </material>
     <!-- BASE LINK -->
