Commit message: slam toolbox changes

File: src/robot-nav/description/robot_core.xacro (robot description, xacro)
@@ -19,6 +19,12 @@
     </material>
     <!-- BASE LINK -->
-    <link name="base_link">
-    </link>
+    <link name="base_link" />
+    <!-- BASE_FOOTPRINT LINK -->
+    <joint name="base_footprint_joint" type="fixed">
+        <parent link="base_link" />
+        <child link="base_footprint" />
+        <origin xyz="0 0 0" rpy="0 0 0" />
+    </joint>
+    <link name="base_footprint" />
     <!-- CHASSIS LINK -->
     <joint name="chassis_joint" type="fixed">

Commit message: xacro updates

File: src/robot-nav/description/robot_core.xacro (robot description, xacro)
@@ -64,5 +64,5 @@
         <visual>
             <geometry>
-                <cylinder radius="0.05" length="0.04" />
+                <cylinder radius="0.02" length="0.04" />
             </geometry>
             <material name="blue" />
@@ -70,8 +70,8 @@
         <collision>
             <geometry>
-                <sphere radius="0.05" />
+                <sphere radius="0.02" />
             </geometry>
         </collision>
-        <xacro:inertial_cylinder mass="0.1" length="0.04" radius="0.05">
+        <xacro:inertial_cylinder mass="0.1" length="0.04" radius="0.02">
             <origin xyz="0 0 0" rpy="0 0 0" />
         </xacro:inertial_cylinder>
@@ -90,5 +90,5 @@
         <visual>
             <geometry>
-                <cylinder radius="0.05" length="0.04" />
+                <cylinder radius="0.02" length="0.04" />
             </geometry>
             <material name="blue" />
@@ -96,8 +96,8 @@
         <collision>
             <geometry>
-                <sphere radius="0.05" />
+                <sphere radius="0.02" />
             </geometry>
         </collision>
-        <xacro:inertial_cylinder mass="0.1" length="0.04" radius="0.05">
+        <xacro:inertial_cylinder mass="0.1" length="0.04" radius="0.02">
             <origin xyz="0 0 0" rpy="0 0 0" />
         </xacro:inertial_cylinder>
@@ -115,5 +115,5 @@
         <visual>
             <geometry>
-                <sphere radius="0.05" />
+                <sphere radius="0.02" />
             </geometry>
             <material name="black" />
@@ -121,8 +121,8 @@
         <collision>
             <geometry>
-                <sphere radius="0.05" />
+                <sphere radius="0.02" />
             </geometry>
         </collision>
-        <xacro:inertial_sphere mass="0.1" radius="0.05">
+        <xacro:inertial_sphere mass="0.1" radius="0.02">
             <origin xyz="0 0 0" rpy="0 0 0" />
         </xacro:inertial_sphere>

File: src/robot-nav/description/ros2_control.xacro (robot description, xacro)
@@ -11,5 +11,5 @@
                 <param name="baud_rate">57600</param>
                 <param name="timeout_ms">1000</param>
-                <param name="enc_counts_per_rev">3436</param>
+                <param name="enc_counts_per_rev">4248</param>
             </hardware>
             <joint name="left_wheel_joint">

Commit message: update params

File: src/robot-nav/description/robot_core.xacro (robot description, xacro)
@@ -28,5 +28,5 @@
     <xacro:property name="chassis_mass" value="1.1" />
     <xacro:property name="wheel_track" value="0.168" />
-    <xacro:property name="wheel_radius" value="0.0368" />
+    <xacro:property name="wheel_radius" value="0.034" />
     <xacro:property name="wheel_length" value="0.0295" />
     <xacro:property name="wheel_mass" value="0.05" />

Commit message: cleanup + ackermann steering

File: src/robot-nav/description/robot_core.xacro (robot description, xacro)
@@ -22,18 +22,26 @@
     </material>
     <!-- VARIABLES-->
-    <xacro:property name="chassis_length" value="0.27" />
+    <xacro:property name="chassis_length"
+        value="0.27" />
     <xacro:property name="chassis_width" value="0.1205" />
-    <xacro:property name="chassis_height" value="0.115" />
-    <xacro:property name="chassis_to_back_wheels_distance" value="0.048" />
+    <xacro:property
+        name="chassis_height" value="0.115" />
+    <xacro:property name="chassis_to_back_wheels_distance"
+        value="0.048" />
     <xacro:property name="chassis_mass" value="1.1" />
-    <xacro:property name="wheel_track" value="0.168" />
-    <xacro:property name="wheel_radius" value="0.034" />
+    <xacro:property
+        name="rear_wheel_track" value="0.175" />
+    <xacro:property name="front_wheel_track"
+        value="0.11" />
+    <xacro:property
+        name="wheel_radius" value="0.034" />
     <xacro:property name="wheel_length" value="0.0295" />
-    <xacro:property name="wheel_mass" value="0.05" />
-    <xacro:property name="wheel_base" value="0.171" />
+    <xacro:property
+        name="wheel_mass" value="0.05" />
+    <xacro:property name="wheel_base" value="0.172" />
     <!-- BASE LINK -->
-    <link name="base_link" />
-    <!-- BASE_FOOTPRINT LINK -->
-    <joint name="base_footprint_joint" type="fixed">
+    <link
+        name="base_link" />
+    <!-- BASE_FOOTPRINT LINK -->Select <joint name="base_footprint_joint" type="fixed">
         <parent link="base_link" />
         <child link="base_footprint" />
@@ -42,5 +50,6 @@
     <link name="base_footprint" />
     <!-- CHASSIS LINK -->
-    <joint name="chassis_joint" type="fixed">
+    <joint
+        name="chassis_joint" type="fixed">
         <parent link="base_link" />
         <child link="chassis" />
@@ -66,12 +75,14 @@
         </xacro:inertial_box>
     </link>
-    <gazebo reference="chassis">
+    <gazebo
+        reference="chassis">
         <material>Gazebo/White</material>
     </gazebo>
     <!-- REAR LEFT WHEEL LINK -->
-    <joint name="rear_left_wheel_joint" type="continuous">
+    <joint name="rear_left_wheel_joint"
+        type="continuous">
         <parent link="base_link" />
         <child link="rear_left_wheel" />
-        <origin xyz="0 ${wheel_track/2} 0" rpy="-${pi/2} 0 0" />
+        <origin xyz="0 ${rear_wheel_track/2} 0" rpy="-${pi/2} 0 0" />
         <axis xyz="0 0 1" />
     </joint>
@@ -93,12 +104,14 @@
         </xacro:inertial_cylinder>
     </link>
-    <gazebo reference="rear_left_wheel">
+    <gazebo
+        reference="rear_left_wheel">
         <material>Gazebo/Blue</material>
     </gazebo>
     <!-- REAR RIGHT WHEEL LINK -->
-    <joint name="rear_right_wheel_joint" type="continuous">
+    <joint name="rear_right_wheel_joint"
+        type="continuous">
         <parent link="base_link" />
         <child link="rear_right_wheel" />
-        <origin xyz="0 -${wheel_track/2} 0" rpy="${pi/2} 0 0" />
+        <origin xyz="0 -${rear_wheel_track/2} 0" rpy="${pi/2} 0 0" />
         <axis xyz="0 0 -1" />
     </joint>
@@ -120,97 +133,68 @@
         </xacro:inertial_cylinder>
     </link>
-    <gazebo reference="rear_right_wheel">
-        <material>Gazebo/Blue</material>
-    </gazebo>
-    <!-- VIRTUAL FRONT WHEEL LINK-->
-    <joint name="virtual_front_wheel_joint" type="revolute">
-        <parent link="base_link" />
-        <child link="virtual_front_wheel" />
-        <origin xyz="${wheel_base} 0.0 0.0" rpy="0 0 ${pi/2}" />
-        <axis xyz="0 0 1" />
-        <limit lower="-0.4" upper="0.4" effort="100.0" velocity="0.0" />
-        <dynamics damping="0.2" />
-    </joint>
-    <link name="virtual_front_wheel">
-        <visual>
-            <origin xyz="0.0 0.0 0.0" rpy="${pi/2} 0 ${pi/2}" />
-            <geometry>
-                <cylinder radius="${wheel_radius}" length="${wheel_length}" />
-            </geometry>
-            <material name="black" />
-        </visual>
-        <collision>
-            <geometry>
-                <sphere radius="${wheel_radius}" />
-            </geometry>
-        </collision>
-        <xacro:inertial_cylinder mass="${wheel_mass}" length="${wheel_length}"
-            radius="${wheel_radius}">
-            <origin xyz="0 0 0" rpy="0 0 0" />
-        </xacro:inertial_cylinder>
-    </link>
-    <gazebo reference="virtual_front_wheel">
-        <material>Gazebo/Blue</material>
-        <mu1 value="0.001" />
-        <mu2 value="0.001" />
+    <gazebo
+        reference="rear_right_wheel">
+        <material>Gazebo/Blue</material>
     </gazebo>
     <!-- FRONT RIGHT WHEEL LINK-->
-    <joint name="front_right_wheel_joint" type="continuous">
+    <joint name="front_right_wheel_joint"
+        type="revolute">
         <parent link="base_link" />
         <child link="front_right_wheel" />
-        <origin xyz="${wheel_base} -${wheel_track/2} 0" rpy="0 0 ${pi/2}" />
+        <origin xyz="${wheel_base} -${front_wheel_track/2} 0" rpy="0 0 ${pi/2}" />
         <axis xyz="0 0 1" />
         <dynamics damping="0.2" />
-        <mimic joint="virtual_front_wheel_joint" multiplier="1.0" offset="0.0" />
-    </joint>
-    <link name="front_right_wheel">
-        <visual>
-            <origin xyz="0.0 0.0 0.0" rpy="${pi/2} 0 ${pi/2}" />
-            <geometry>
-                <cylinder radius="${wheel_radius}" length="${wheel_length}" />
-            </geometry>
-            <material name="blue" />
-        </visual>
-        <collision>
-            <geometry>
-                <sphere radius="${wheel_radius}" />
-            </geometry>
-        </collision>
-        <xacro:inertial_cylinder mass="${wheel_mass}" length="${wheel_length}"
-            radius="${wheel_radius}">
-            <origin xyz="0 0 0" rpy="0 0 0" />
-        </xacro:inertial_cylinder>
-    </link>
-    <gazebo reference="front_right_wheel">
-        <material>Gazebo/Blue</material>
-    </gazebo>
+        <limit lower="-0.41" upper="0.47" effort="100.0" velocity="0.0" />
+    </joint>
+    <link
+        name="front_right_wheel">
+        <visual>
+            <origin xyz="-0.0325 0.0 0.0" rpy="${pi/2} 0 ${pi/2}" />
+            <geometry>
+                <cylinder radius="${wheel_radius}" length="${wheel_length}" />
+            </geometry>
+            <material name="blue" />
+        </visual>
+        <collision>
+            <geometry>
+                <sphere radius="${wheel_radius}" />
+            </geometry>
+        </collision>
+        <xacro:inertial_cylinder mass="${wheel_mass}" length="${wheel_length}"
+            radius="${wheel_radius}">
+            <origin xyz="-0.0325 0.0 0" rpy="0 0 0" />
+        </xacro:inertial_cylinder>
+    </link>
     <!-- FRONT LEFT WHEEL LINK-->
-    <joint name="front_left_wheel_joint" type="continuous">
+    <joint
+        name="front_left_wheel_joint" type="revolute">
         <parent link="base_link" />
         <child link="front_left_wheel" />
-        <origin xyz="${wheel_base} ${wheel_track/2} 0" rpy="0 0 ${pi/2}" />
+        <origin xyz="${wheel_base} ${front_wheel_track/2} 0" rpy="0 0 ${pi/2}" />
         <axis xyz="0 0 1" />
         <dynamics damping="0.2" />
-        <mimic joint="virtual_front_wheel_joint" multiplier="1.0" offset="0.0" />
-    </joint>
-    <link name="front_left_wheel">
-        <visual>
-            <origin xyz="0.0 0.0 0.0" rpy="${pi/2} 0 ${pi/2}" />
-            <geometry>
-                <cylinder radius="${wheel_radius}" length="${wheel_length}" />
-            </geometry>
-            <material name="blue" />
-        </visual>
-        <collision>
-            <geometry>
-                <sphere radius="${wheel_radius}" />
-            </geometry>
-        </collision>
-        <xacro:inertial_cylinder mass="${wheel_mass}" length="${wheel_length}"
-            radius="${wheel_radius}">
-            <origin xyz="0 0 0" rpy="0 0 0" />
-        </xacro:inertial_cylinder>
-    </link>
-    <gazebo reference="front_left_wheel">
+        <limit lower="-0.38" upper="0.54" effort="100.0" velocity="0.0" />
+    </joint>
+    <link
+        name="front_left_wheel">
+        <visual>
+            <origin xyz="0.0325 0.0 0.0" rpy="${pi/2} 0 ${pi/2}" />
+            <geometry>
+                <cylinder radius="${wheel_radius}" length="${wheel_length}" />
+            </geometry>
+            <material name="blue" />
+        </visual>
+        <collision>
+            <geometry>
+                <sphere radius="${wheel_radius}" />
+            </geometry>
+        </collision>
+        <xacro:inertial_cylinder mass="${wheel_mass}" length="${wheel_length}"
+            radius="${wheel_radius}">
+            <origin xyz="0.0325 0.0 0.0" rpy="0 0 0" />
+        </xacro:inertial_cylinder>
+    </link>
+    <gazebo
+        reference="front_left_wheel">
         <material>Gazebo/Blue</material>
     </gazebo>
@@ -218,30 +202,3 @@
         <material>Gazebo/Blue</material>
     </gazebo>
-    <!-- CASTER WHEEL LINK-->
-    <!-- <joint name="caster_wheel_joint" type="fixed">
-        <parent link="chassis" />
-        <child link="caster_wheel" />
-        <origin xyz="0.24 0.0 0.0" />
-    </joint>
-    <link name="caster_wheel">
-        <visual>
-            <geometry>
-                <sphere radius="0.02" />
-            </geometry>
-            <material name="black" />
-        </visual>
-        <collision>
-            <geometry>
-                <sphere radius="0.02" />
-            </geometry>
-        </collision>
-        <xacro:inertial_sphere mass="0.1" radius="0.02">
-            <origin xyz="0 0 0" rpy="0 0 0" />
-        </xacro:inertial_sphere>
-    </link>
-    <gazebo reference="caster_wheel">
-        <material>Gazebo/Black</material>
-        <mu1 value="0.001" />
-        <mu2 value="0.001" />
-    </gazebo> -->
 </robot>

File: src/robot-nav/description/ros2_control.xacro (robot description, xacro)
@@ -3,6 +3,7 @@
     <ros2_control name="RealRobot" type="system">
         <hardware>
-            <plugin>tricycle_arduino/TricycleArduinoHardware</plugin>
-            <param name="front_wheel_name">virtual_front_wheel_joint</param>
+            <plugin>ackermann_arduino/AckermannArduinoHardware</plugin>
+            <param name="front_left_wheel_name">front_left_wheel_joint</param>
+            <param name="front_right_wheel_name">front_right_wheel_joint</param>
             <param name="rear_left_wheel_name">rear_left_wheel_joint</param>
             <param name="rear_right_wheel_name">rear_right_wheel_joint</param>
@@ -13,5 +14,9 @@
             <param name="enc_counts_per_rev">1320</param>
         </hardware>
-        <joint name="virtual_front_wheel_joint">
+        <joint name="front_left_wheel_joint">
+            <command_interface name="position" />
+            <state_interface name="position" />
+        </joint>
+        <joint name="front_right_wheel_joint">
             <command_interface name="position" />
             <state_interface name="position" />
