Commit message: tricycle

File: src/robot-nav/description/lidar.xacro (robot description, xacro)
@@ -4,5 +4,5 @@
         <parent link="chassis" />
         <child link="laser_frame" />
-        <origin xyz="0.1 0.0 0.175" rpy="0.0 0.0 0.0" />
+        <origin xyz="0.23 0.0 0.175" rpy="0.0 0.0 0.0" />
     </joint>
     <link name="laser_frame">

File: src/robot-nav/description/robot.urdf.xacro (robot description, xacro)
@@ -4,12 +4,7 @@
     <xacro:arg name="sim_mode" default="false" />
     <xacro:include filename="robot_core.xacro" />
-    <xacro:if value="$(arg use_ros2_control)">
-        <xacro:include filename="ros2_control.xacro" />
-    </xacro:if>
-    <xacro:unless value="$(arg use_ros2_control)">
-        <xacro:include filename="gazebo_control.xacro" />
-    </xacro:unless>
-    <xacro:include filename="lidar.xacro" />
+    <xacro:include filename="ros2_control.xacro" />
+    <!-- <xacro:include filename="lidar.xacro" /> -->
     <!-- <xacro:include filename="camera.xacro" /> -->
-    <xacro:include filename="depth_camera.xacro" />
+    <!-- <xacro:include filename="depth_camera.xacro" /> -->
 </robot>

File: src/robot-nav/description/robot_core.xacro (robot description, xacro)
@@ -18,4 +18,18 @@
         <color rgba="1.0 0.0 0.0 1.0" />
     </material>
+    <material name="invisible">
+        <color rgba="1.0 1.0 1.0 0.0" />
+    </material>
+    <!-- VARIABLES-->
+    <xacro:property name="chassis_length" value="0.27" />
+    <xacro:property name="chassis_width" value="0.1205" />
+    <xacro:property name="chassis_height" value="0.115" />
+    <xacro:property name="chassis_to_back_wheels_distance" value="0.048" />
+    <xacro:property name="chassis_mass" value="1.1" />
+    <xacro:property name="wheel_track" value="0.168" />
+    <xacro:property name="wheel_radius" value="0.0368" />
+    <xacro:property name="wheel_length" value="0.0295" />
+    <xacro:property name="wheel_mass" value="0.05" />
+    <xacro:property name="wheel_base" value="0.171" />
     <!-- BASE LINK -->
     <link name="base_link" />
@@ -31,22 +45,23 @@
         <parent link="base_link" />
         <child link="chassis" />
-        <origin xyz="-0.1 0.0 0.0" />
+        <origin xyz="-${chassis_to_back_wheels_distance} 0.0 0.0" />
     </joint>
     <link name="chassis">
         <visual>
-            <origin xyz="0.15 0.0 0.075" />
-            <geometry>
-                <box size="0.3 0.3 0.15" />
+            <origin xyz="${chassis_length/2} 0.0 ${chassis_height/3}" />
+            <geometry>
+                <box size="${chassis_length} ${chassis_width} ${chassis_height}" />
             </geometry>
             <material name="white" />
         </visual>
         <collision>
-            <origin xyz="0.15 0.0 0.075" />
-            <geometry>
-                <box size="0.3 0.3 0.15" />
-            </geometry>
-        </collision>
-        <xacro:inertial_box mass="0.5" x="0.3" y="0.3" z="0.15">
-            <origin xyz="0.15 0 0.075" />
+            <origin xyz="${chassis_length/2} 0.0 ${chassis_height/3}" />
+            <geometry>
+                <box size="${chassis_length} ${chassis_width} ${chassis_height}" />
+            </geometry>
+        </collision>
+        <xacro:inertial_box mass="${chassis_mass}" x="${chassis_length}" y="${chassis_width}"
+            z="${chassis_height}">
+            <origin xyz="0.0 0 0.0" />
         </xacro:inertial_box>
     </link>
@@ -54,58 +69,155 @@
         <material>Gazebo/White</material>
     </gazebo>
-    <!-- LEFT WHEEL LINK -->
-    <joint name="left_wheel_joint" type="continuous">
-        <parent link="base_link" />
-        <child link="left_wheel" />
-        <origin xyz="0 0.175 0" rpy="-${pi/2} 0 0" />
-        <axis xyz="0 0 1" />
-    </joint>
-    <link name="left_wheel">
-        <visual>
-            <geometry>
-                <cylinder radius="0.02" length="0.04" />
-            </geometry>
-            <material name="blue" />
-        </visual>
-        <collision>
-            <geometry>
-                <sphere radius="0.02" />
-            </geometry>
-        </collision>
-        <xacro:inertial_cylinder mass="0.1" length="0.04" radius="0.02">
-            <origin xyz="0 0 0" rpy="0 0 0" />
-        </xacro:inertial_cylinder>
-    </link>
-    <gazebo reference="left_wheel">
-        <material>Gazebo/Blue</material>
-    </gazebo>
-    <!-- RIGHT WHEEL LINK -->
-    <joint name="right_wheel_joint" type="continuous">
-        <parent link="base_link" />
-        <child link="right_wheel" />
-        <origin xyz="0 -0.175 0" rpy="${pi/2} 0 0" />
+    <!-- REAR LEFT WHEEL LINK -->
+    <joint name="rear_left_wheel_joint" type="continuous">
+        <parent link="base_link" />
+        <child link="rear_left_wheel" />
+        <origin xyz="0 ${wheel_track/2} 0" rpy="-${pi/2} 0 0" />
+        <axis xyz="0 0 1" />
+    </joint>
+    <link name="rear_left_wheel">
+        <visual>
+            <geometry>
+                <cylinder radius="${wheel_radius}" length="${wheel_length}" />
+            </geometry>
+            <material name="blue" />
+        </visual>
+        <collision>
+            <geometry>
+                <sphere radius="${wheel_radius}" />
+            </geometry>
+        </collision>
+        <xacro:inertial_cylinder mass="${wheel_mass}" length="${wheel_length}"
+            radius="${wheel_radius}">
+            <origin xyz="0 0 0" rpy="0 0 0" />
+        </xacro:inertial_cylinder>
+    </link>
+    <gazebo reference="rear_left_wheel">
+        <material>Gazebo/Blue</material>
+    </gazebo>
+    <!-- REAR RIGHT WHEEL LINK -->
+    <joint name="rear_right_wheel_joint" type="continuous">
+        <parent link="base_link" />
+        <child link="rear_right_wheel" />
+        <origin xyz="0 -${wheel_track/2} 0" rpy="${pi/2} 0 0" />
         <axis xyz="0 0 -1" />
     </joint>
-    <link name="right_wheel">
-        <visual>
-            <geometry>
-                <cylinder radius="0.02" length="0.04" />
-            </geometry>
-            <material name="blue" />
-        </visual>
-        <collision>
-            <geometry>
-                <sphere radius="0.02" />
-            </geometry>
-        </collision>
-        <xacro:inertial_cylinder mass="0.1" length="0.04" radius="0.02">
-            <origin xyz="0 0 0" rpy="0 0 0" />
-        </xacro:inertial_cylinder>
-    </link>
-    <gazebo reference="right_wheel">
+    <link name="rear_right_wheel">
+        <visual>
+            <geometry>
+                <cylinder radius="${wheel_radius}" length="${wheel_length}" />
+            </geometry>
+            <material name="blue" />
+        </visual>
+        <collision>
+            <geometry>
+                <sphere radius="${wheel_radius}" />
+            </geometry>
+        </collision>
+        <xacro:inertial_cylinder mass="${wheel_mass}" length="${wheel_length}"
+            radius="${wheel_radius}">
+            <origin xyz="0 0 0" rpy="0 0 0" />
+        </xacro:inertial_cylinder>
+    </link>
+    <gazebo reference="rear_right_wheel">
+        <material>Gazebo/Blue</material>
+    </gazebo>
+    <!-- VIRTUAL FRONT WHEEL LINK-->
+    <joint name="virtual_front_wheel_joint" type="revolute">
+        <parent link="base_link" />
+        <child link="virtual_front_wheel" />
+        <origin xyz="${wheel_base} 0.0 0.0" rpy="0 0 ${pi/2}" />
+        <axis xyz="0 0 1" />
+        <limit lower="-0.4" upper="0.4" effort="100.0" velocity="0.0" />
+        <dynamics damping="0.2" />
+    </joint>
+    <link name="virtual_front_wheel">
+        <visual>
+            <origin xyz="0.0 0.0 0.0" rpy="${pi/2} 0 ${pi/2}" />
+            <geometry>
+                <cylinder radius="${wheel_radius}" length="${wheel_length}" />
+            </geometry>
+            <material name="black" />
+        </visual>
+        <collision>
+            <geometry>
+                <sphere radius="${wheel_radius}" />
+            </geometry>
+        </collision>
+        <xacro:inertial_cylinder mass="${wheel_mass}" length="${wheel_length}"
+            radius="${wheel_radius}">
+            <origin xyz="0 0 0" rpy="0 0 0" />
+        </xacro:inertial_cylinder>
+    </link>
+    <gazebo reference="virtual_front_wheel">
+        <material>Gazebo/Blue</material>
+        <mu1 value="0.001" />
+        <mu2 value="0.001" />
+    </gazebo>
+    <!-- FRONT RIGHT WHEEL LINK-->
+    <joint name="front_right_wheel_joint" type="continuous">
+        <parent link="base_link" />
+        <child link="front_right_wheel" />
+        <origin xyz="${wheel_base} -${wheel_track/2} 0" rpy="0 0 ${pi/2}" />
+        <axis xyz="0 0 1" />
+        <dynamics damping="0.2" />
+        <mimic joint="virtual_front_wheel_joint" multiplier="1.0" offset="0.0" />
+    </joint>
+    <link name="front_right_wheel">
+        <visual>
+            <origin xyz="0.0 0.0 0.0" rpy="${pi/2} 0 ${pi/2}" />
+            <geometry>
+                <cylinder radius="${wheel_radius}" length="${wheel_length}" />
+            </geometry>
+            <material name="blue" />
+        </visual>
+        <collision>
+            <geometry>
+                <sphere radius="${wheel_radius}" />
+            </geometry>
+        </collision>
+        <xacro:inertial_cylinder mass="${wheel_mass}" length="${wheel_length}"
+            radius="${wheel_radius}">
+            <origin xyz="0 0 0" rpy="0 0 0" />
+        </xacro:inertial_cylinder>
+    </link>
+    <gazebo reference="front_right_wheel">
+        <material>Gazebo/Blue</material>
+    </gazebo>
+    <!-- FRONT LEFT WHEEL LINK-->
+    <joint name="front_left_wheel_joint" type="continuous">
+        <parent link="base_link" />
+        <child link="front_left_wheel" />
+        <origin xyz="${wheel_base} ${wheel_track/2} 0" rpy="0 0 ${pi/2}" />
+        <axis xyz="0 0 1" />
+        <dynamics damping="0.2" />
+        <mimic joint="virtual_front_wheel_joint" multiplier="1.0" offset="0.0" />
+    </joint>
+    <link name="front_left_wheel">
+        <visual>
+            <origin xyz="0.0 0.0 0.0" rpy="${pi/2} 0 ${pi/2}" />
+            <geometry>
+                <cylinder radius="${wheel_radius}" length="${wheel_length}" />
+            </geometry>
+            <material name="blue" />
+        </visual>
+        <collision>
+            <geometry>
+                <sphere radius="${wheel_radius}" />
+            </geometry>
+        </collision>
+        <xacro:inertial_cylinder mass="${wheel_mass}" length="${wheel_length}"
+            radius="${wheel_radius}">
+            <origin xyz="0 0 0" rpy="0 0 0" />
+        </xacro:inertial_cylinder>
+    </link>
+    <gazebo reference="front_left_wheel">
+        <material>Gazebo/Blue</material>
+    </gazebo>
+    <gazebo reference="front_left_wheel_joint">
         <material>Gazebo/Blue</material>
     </gazebo>
     <!-- CASTER WHEEL LINK-->
-    <joint name="caster_wheel_joint" type="fixed">
+    <!-- <joint name="caster_wheel_joint" type="fixed">
         <parent link="chassis" />
         <child link="caster_wheel" />
@@ -132,4 +244,4 @@
         <mu1 value="0.001" />
         <mu2 value="0.001" />
-    </gazebo>
+    </gazebo> -->
 </robot>

File: src/robot-nav/description/ros2_control.xacro (robot description, xacro)
@@ -1,62 +1,30 @@
 <?xml version="1.0"?>
 <robot xmlns:xacro="http://www.ros.org/wiki/xacro">
-    <xacro:unless value="$(arg sim_mode)">
-        <ros2_control name="RealRobot" type="system">
-            <hardware>
-                <plugin>diffdrive_arduino/DiffDriveArduinoHardware</plugin>
-                <param name="left_wheel_name">left_wheel_joint</param>
-                <param name="right_wheel_name">right_wheel_joint</param>
-                <param name="loop_rate">30</param>
-                <param name="device">/dev/ttyACM0</param>
-                <param name="baud_rate">57600</param>
-                <param name="timeout_ms">1000</param>
-                <param name="enc_counts_per_rev">4248</param>
-            </hardware>
-            <joint name="left_wheel_joint">
-                <command_interface name="velocity">
-                    <param name="min">-10</param>
-                    <param name="max">10</param>
-                </command_interface>
-                <state_interface name="position"></state_interface>
-                <state_interface name="velocity"></state_interface>
-            </joint>
-            <joint name="right_wheel_joint">
-                <command_interface name="velocity">
-                    <param name="min">-10</param>
-                    <param name="max">10</param>
-                </command_interface>
-                <state_interface name="position"></state_interface>
-                <state_interface name="velocity"></state_interface>
-            </joint>
-        </ros2_control>
-    </xacro:unless>
-    <xacro:if value="$(arg sim_mode)">
-        <ros2_control name="GazeboSystem" type="system">
-            <hardware>
-                <plugin>gazebo_ros2_control/GazeboSystem</plugin>
-            </hardware>
-            <joint name="left_wheel_joint">
-                <command_interface name="velocity">
-                    <param name="min">-10</param>
-                    <param name="max">10</param>
-                </command_interface>
-                <state_interface name="velocity"></state_interface>
-                <state_interface name="position"></state_interface>
-            </joint>
-            <joint name="right_wheel_joint">
-                <command_interface name="velocity">
-                    <param name="min">-10</param>
-                    <param name="max">10</param>
-                </command_interface>
-                <state_interface name="velocity"></state_interface>
-                <state_interface name="position"></state_interface>
-            </joint>
-        </ros2_control>
-    </xacro:if>
-    <gazebo>
-        <plugin name="gazebo_ros2_control" filename="libgazebo_ros2_control.so">
-            <parameters>$(find robot-nav)/config/my_controllers.yaml</parameters>
-            <parameters>$(find robot-nav)/config/gaz_ros2_ctl_use_sim.yaml</parameters>
-        </plugin>
-    </gazebo>
+    <ros2_control name="RealRobot" type="system">
+        <hardware>
+            <plugin>tricycle_arduino/TricycleArduinoHardware</plugin>
+            <param name="front_wheel_name">virtual_front_wheel_joint</param>
+            <param name="rear_left_wheel_name">rear_left_wheel_joint</param>
+            <param name="rear_right_wheel_name">rear_right_wheel_joint</param>
+            <param name="loop_rate">30</param>
+            <param name="device">/dev/ttyACM0</param>
+            <param name="baud_rate">57600</param>
+            <param name="timeout_ms">1000</param>
+            <param name="enc_counts_per_rev">1320</param>
+        </hardware>
+        <joint name="virtual_front_wheel_joint">
+            <command_interface name="position" />
+            <state_interface name="position" />
+        </joint>
+        <joint name="rear_left_wheel_joint">
+            <command_interface name="velocity" />
+            <state_interface name="velocity" />
+            <state_interface name="position" />
+        </joint>
+        <joint name="rear_right_wheel_joint">
+            <command_interface name="velocity" />
+            <state_interface name="velocity" />
+            <state_interface name="position" />
+        </joint>
+    </ros2_control>
 </robot>

Commit message: twistmux

File: src/robot-nav/description/lidar.xacro (robot description, xacro)
@@ -4,5 +4,5 @@
         <parent link="chassis" />
         <child link="laser_frame" />
-        <origin xyz="0.23 0.0 0.175" rpy="0.0 0.0 0.0" />
+        <origin xyz="0.105 0.0 0.135" rpy="0.0 0.0 0.0" />
     </joint>
     <link name="laser_frame">

File: src/robot-nav/description/robot.urdf.xacro (robot description, xacro)
@@ -5,5 +5,5 @@
     <xacro:include filename="robot_core.xacro" />
     <xacro:include filename="ros2_control.xacro" />
-    <!-- <xacro:include filename="lidar.xacro" /> -->
+    <xacro:include filename="lidar.xacro" />
     <!-- <xacro:include filename="camera.xacro" /> -->
     <!-- <xacro:include filename="depth_camera.xacro" /> -->

Commit message: imu

File: src/robot-nav/description/lidar.xacro (robot description, xacro)
@@ -4,5 +4,5 @@
         <parent link="chassis" />
         <child link="laser_frame" />
-        <origin xyz="0.105 0.0 0.135" rpy="0.0 0.0 0.0" />
+        <origin xyz="0.107 0.0 0.135" rpy="0.0 0.0 0.0" />
     </joint>
     <link name="laser_frame">

File: src/robot-nav/description/robot.urdf.xacro (robot description, xacro)
@@ -6,4 +6,5 @@
     <xacro:include filename="ros2_control.xacro" />
     <xacro:include filename="lidar.xacro" />
+    <xacro:include filename="imu.xacro" />
     <!-- <xacro:include filename="camera.xacro" /> -->
     <!-- <xacro:include filename="depth_camera.xacro" /> -->
