Commit message: changes

File: src/robot-nav/description/camera.xacro (robot description, xacro)
@@ -4,5 +4,5 @@
         <parent link="chassis" />
         <child link="camera_link" />
-        <origin xyz="0.305 0.0 0.08" rpy="0.0 0.0 0.0" />
+        <origin xyz="0.24 0.0 0.13" rpy="0.0 0.0 0.0" />
     </joint>
     <link name="camera_link">
@@ -14,32 +14,3 @@
         </visual>
     </link>
-    <joint name="camera_optical_joint" type="fixed">
-        <parent link="camera_link" />
-        <child link="camera_link_optical" />
-        <origin xyz="0.0 0.0 0.0" rpy="${-pi/2} 0.0 ${-pi/2}" />
-    </joint>
-    <link name="camera_link_optical" />
-    <gazebo reference="camera_link">
-        <material>Gazebo/Red</material>
-        <sensor name="camera" type="camera">
-            <pose> 0 0 0 0 0 0 </pose>
-            <visualize>true</visualize>
-            <update_rate>10</update_rate>
-            <camera>
-                <horizontal_fov>1.204</horizontal_fov>
-                <image>
-                    <format>R8G8B8</format>
-                    <width>640</width>
-                    <height>480</height>
-                </image>
-                <clip>
-                    <near>0.05</near>
-                    <far>8.0</far>
-                </clip>
-            </camera>
-            <plugin name="camera_controller" filename="libgazebo_ros_camera.so">
-                <frame_name>camera_link_optical</frame_name>
-            </plugin>
-        </sensor>
-    </gazebo>
 </robot>

File: src/robot-nav/description/lidar.xacro (robot description, xacro)
@@ -4,5 +4,5 @@
         <parent link="chassis" />
         <child link="laser_frame" />
-        <origin xyz="0.107 0.0 0.135" rpy="0.0 0.0 0.0" />
+        <origin xyz="0.175 0.0 0.153" rpy="0.0 0.0 0.0" />
     </joint>
     <link name="laser_frame">

File: src/robot-nav/description/robot.urdf.xacro (robot description, xacro)
@@ -7,5 +7,5 @@
     <xacro:include filename="lidar.xacro" />
     <xacro:include filename="imu.xacro" />
-    <!-- <xacro:include filename="camera.xacro" /> -->
+    <xacro:include filename="camera.xacro" />
     <!-- <xacro:include filename="depth_camera.xacro" /> -->
 </robot>

File: src/robot-nav/description/robot_core.xacro (robot description, xacro)
@@ -145,5 +145,5 @@
         <axis xyz="0 0 1" />
         <dynamics damping="0.2" />
-        <limit lower="-0.41" upper="0.47" effort="100.0" velocity="0.0" />
+        <limit lower="-0.454" upper="0.384" effort="100.0" velocity="0.0" />
     </joint>
     <link
@@ -174,5 +174,5 @@
         <axis xyz="0 0 1" />
         <dynamics damping="0.2" />
-        <limit lower="-0.38" upper="0.54" effort="100.0" velocity="0.0" />
+        <limit lower="-0.384" upper="0.454" effort="100.0" velocity="0.0" />
     </joint>
     <link

File: src/robot-nav/description/ros2_control.xacro (robot description, xacro)
@@ -10,5 +10,5 @@
             <param name="loop_rate">30</param>
             <param name="device">/dev/ttyACM0</param>
-            <param name="baud_rate">57600</param>
+            <param name="baud_rate">115200</param>
             <param name="timeout_ms">1000</param>
             <param name="enc_counts_per_rev">1320</param>
