Commit message: imu model changed

File: src/robot-nav/description/imu.xacro (robot description, xacro)
@@ -4,5 +4,5 @@
         <parent link="chassis" />
         <child link="imu_link" />
-        <origin xyz="${chassis_to_back_wheels_distance} 0.05 0.0" rpy="0.0 0.0 0.0" />
+        <origin xyz="0.208 0.03 0.0" rpy="0.0 0.0 0.0" />
     </joint>
     <link name="imu_link">
